File: EAGLE/Nick Lester Final.brd (EAGLE design)
At the start: 88.9 x 50.8 mm, 13 parts, among them U1 POCKETBEAGLE, U2 0.56_HEX_BACKPACK

Commit message: Add files via upload
Parts:
- added FUD1, FUD2, FUD3: FIDUCIAL, ENGI301:FIDUCIAL_40MIL
Changed lines of the file:
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@@
 <layer number="21" name="tPlace" color="7" fill="1" visible="yes" active="yes"/>
 <layer number="22" name="bPlace" color="7" fill="1" visible="yes" active="yes"/>
-<layer number="23" name="tOrigins" color="15" fill="1" visible="no" active="yes"/>
-<layer number="24" name="bOrigins" color="15" fill="1" visible="no" active="yes"/>
+<layer number="23" name="tOrigins" color="15" fill="1" visible="yes" active="yes"/>
+<layer number="24" name="bOrigins" color="15" fill="1" visible="yes" active="yes"/>
 <layer number="25" name="tNames" color="7" fill="1" visible="yes" active="yes"/>
 <layer number="26" name="bNames" color="7" fill="1" visible="yes" active="yes"/>
@@
 </element>
 <element name="BUZZER_1" library="Nick Lester Final" package="PS1240_BUZZER" value="PS1240_BUZZER" x="80.01" y="40.64" smashed="yes">
-<attribute name="NAME" x="73.11" y="48.04" size="1.27" layer="21" font="vector"/>
+<attribute name="NAME" x="73.745" y="48.04" size="1.27" layer="21" font="vector"/>
 </element>
 <element name="BUZZER_2" library="Nick Lester Final" package="PS1240_BUZZER" value="PS1240_BUZZER" x="8.89" y="40.64" smashed="yes">
-<attribute name="NAME" x="1.99" y="48.04" size="1.27" layer="21" font="vector"/>
+<attribute name="NAME" x="2.625" y="48.04" size="1.27" layer="21" font="vector"/>
 </element>
 <element name="BARREL_CONNECTOR" library="Nick Lester Final" package="BARREL_CONNECTOR" value="BARREL_CONNECTOR" x="7.493" y="12.065" smashed="yes" rot="MR180">
 <attribute name="NAME" x="13.863" y="11.775" size="0.762" layer="22" font="vector" rot="MR270"/>
 </element>
+<element name="FUD1" library="ENGI301" package="FIDUCIAL_40MIL" value="FIDUCIAL" x="87.63" y="49.53" smashed="yes"/>
+<element name="FUD2" library="ENGI301" package="FIDUCIAL_40MIL" value="FIDUCIAL" x="17.145" y="1.27" smashed="yes"/>
+<element name="FUD3" library="ENGI301" package="FIDUCIAL_40MIL" value="FIDUCIAL" x="87.63" y="1.27" smashed="yes"/>
 </elements>
 <signals>
