File: EAGLE/Nick Lester Final.sch (EAGLE design)
At the start: 13 parts, among them U1 POCKETBEAGLE, U2 0.56_HEX_BACKPACK

Commit message: Add files via upload
Parts:
- added FUD1, FUD2, FUD3: FIDUCIAL, ENGI301:FIDUCIAL
Other:
- note added: "Mechanical"
Changed lines of the file:
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@@
 <part name="BARREL_CONNECTOR" library="Nick Lester Final" deviceset="BARREL_CONNECTOR" device=""/>
 <part name="GND10" library="ENGI301" deviceset="GND" device=""/>
+<part name="FUD1" library="ENGI301" deviceset="FIDUCIAL" device=""/>
+<part name="FUD2" library="ENGI301" deviceset="FIDUCIAL" device=""/>
+<part name="FUD3" library="ENGI301" deviceset="FIDUCIAL" device=""/>
 </parts>
 <sheets>
@@
 <wire x1="5.08" y1="60.96" x2="135.89" y2="60.96" width="0.1524" layer="97"/>
 <text x="11.43" y="48.26" size="6.4516" layer="97">Power Source</text>
+<wire x1="138.43" y1="60.96" x2="260.35" y2="60.96" width="0.1524" layer="97"/>
+<text x="143.51" y="49.53" size="6.4516" layer="97">Mechanical</text>
 </plain>
 <instances>
@@
 <attribute name="VALUE" x="106.68" y="17.78" size="1.778" layer="96" rot="R90"/>
 </instance>
+<instance part="FUD1" gate="G$1" x="162.56" y="34.29" smashed="yes"/>
+<instance part="FUD2" gate="G$1" x="175.26" y="34.29" smashed="yes"/>
+<instance part="FUD3" gate="G$1" x="186.69" y="34.29" smashed="yes"/>
 </instances>
 <busses>
